Commit message: Add black parts (motor, cables, ...) of TriFingerPro
Since pyBullet doesn't support visuals with different materials on the
same link, add the black parts as separate fixed links.

File: xacro/pro/fingerpro.urdf.xacro (robot description, xacro)
@@ -9,12 +9,9 @@
     -->
     <xacro:include filename="fingerpro_macro.xacro" />
-    <material name="finger_material">
-        <color rgba="0.6 0.6 0.6 1.0" />
-    </material>
     <!--
     Simply calling the "finger" macro (without passing any suffix) implies a call for single finger.
     The parameters are automatically set inside the finger_macro file, to accomodate for single finger.
     -->
-    <xacro:fingerpro material="finger_material" />
+    <xacro:fingerpro />
     <!--
     Define the global base link and place the finger relative to it.
@@ -23,9 +20,9 @@
     <link name="center_link">
         <xacro:add_geometry
-                        rpy="0 0 0"
-                        xyz="0 0 0"
-                        mesh_file="${center_link_mesh}"
-                        material="finger_material"
-                        mesh_scale="1." />
+            rpy="0 0 0"
+            xyz="0 0 0"
+            mesh_file="${center_link_mesh}"
+            mesh_scale="1."
+            material="fingerpro_shell"/>
         <xacro:add_inertia
             length_x="0.005"

File: xacro/pro/fingerpro_macro.xacro (robot description, xacro)
@@ -18,4 +18,5 @@
     <xacro:property name="lower_link_mesh" value="${mesh_dir}/SIM__BL-Finger_Tip_without_tip.${mesh_file_extension}"/>
     <xacro:property name="tip_link_mesh" value="${mesh_dir}/SIM__BL-Finger_Tip_actual_tip.${mesh_file_extension}"/>
+    <xacro:property name="motor_mesh" value="${mesh_dir}/SIM__BL-Finger_Motor.dae"/>
     <!-- Distance from outer edge of the link to the joint center -->
     <xacro:property name="upper_link_length" value="0.20945" />
@@ -28,4 +29,10 @@
     <xacro:property name="mesh_x_offset" value="0.014" />
     <xacro:property name="lower_joint_to_tip_distance" value="0.1626" />
+    <material name="fingerpro_shell">
+        <color rgba="0.83 0.79 0.82 1.0" />
+    </material>
+    <material name="fingerpro_motor">
+        <color rgba="0.1 0.1 0.1 1.0" />
+    </material>
     <!--
     Defining the "finger" macro which is used for both single and tri-finger.
@@ -33,5 +40,5 @@
     In case of single finger, no "suffix" value is passed.
     -->
-    <xacro:macro name="fingerpro" params="material suffix:=''">
+    <xacro:macro name="fingerpro" params="suffix:=''">
         <!--
         Fixed links for the finger base (parts where the upper link is mounted).
@@ -43,5 +50,5 @@
                 xyz="0 ${upper_link_length+center_offset} 0"
                 mesh_file="${upper_base_mesh}"
-                material="${material}"
+                material="fingerpro_shell"
                 mesh_scale="1." />
             <xacro:add_inertia
@@ -57,5 +64,5 @@
                 xyz="0 ${center_offset} 0"
                 mesh_file="${upper_link_mesh}"
-                material="${material}"
+                material="fingerpro_shell"
                 mesh_scale="1." />
             <xacro:add_inertia
@@ -66,4 +73,43 @@
                 com="0 0.06 0"/>
         </link>
+        <link name="finger_upper_link_motor${suffix}">
+            <!-- motor -->
+            <visual>
+                <origin xyz="0.018 0.141 -0.001" />
+                <geometry>
+                    <mesh filename="${motor_mesh}"/>
+                </geometry>
+                <material name="fingerpro_motor" />
+            </visual>
+            <!-- end stop -->
+            <visual>
+                <origin xyz="0.015 0.06 0" rpy="0 ${pi/2} 0" />
+                <geometry>
+                    <cylinder length="0.01" radius="0.005"/>
+                </geometry>
+                <material name="fingerpro_motor" />
+            </visual>
+            <!-- cables -->
+            <visual>
+                <origin xyz="-0.008 0.1 0" rpy="${pi/2} 0 0" />
+                <geometry>
+                    <cylinder length="0.12" radius="0.002"/>
+                </geometry>
+                <material name="fingerpro_motor" />
+            </visual>
+            <!-- opening on lower joint -->
+            <visual>
+                <origin xyz="-0.008 0.026 0" rpy="0 ${pi/2} 0" />
+                <geometry>
+                    <cylinder length="0.002" radius="0.014"/>
+                </geometry>
+                <material name="fingerpro_motor" />
+            </visual>
+        </link>
+        <joint name="finger_upper_to_motor_joint${suffix}" type="fixed">
+            <parent link="finger_upper_link${suffix}"/>
+            <child link="finger_upper_link_motor${suffix}"/>
+            <origin xyz="0 ${center_offset} 0" />
+        </joint>
         <link name="finger_middle_link${suffix}">
             <xacro:add_geometry
@@ -71,5 +117,5 @@
                 xyz="0 0 0"
                 mesh_file="${middle_link_mesh}"
-                material="${material}"
+                material="fingerpro_shell"
                 mesh_scale="1." />
             <xacro:add_inertia
@@ -80,4 +126,42 @@
                 com="${2 * mesh_x_offset} 0 -0.08"/>
         </link>
+        <link name="finger_middle_link_motor${suffix}">
+            <!-- motor -->
+            <visual>
+                <origin xyz="0.048 0 -0.046" />
+                <geometry>
+                    <mesh filename="${motor_mesh}"/>
+                </geometry>
+                <material name="fingerpro_motor" />
+            </visual>
+            <!-- end stop -->
+            <visual>
+                <origin xyz="0.048 0 -0.13" rpy="0 ${pi/2} 0" />
+                <geometry>
+                    <cylinder length="0.01" radius="0.005"/>
+                </geometry>
+                <material name="fingerpro_motor" />
+            </visual>
+            <!-- cables -->
+            <visual>
+                <origin xyz="0.025 0 -0.09" />
+                <geometry>
+                    <cylinder length="0.12" radius="0.002"/>
+                </geometry>
+                <material name="fingerpro_motor" />
+            </visual>
+            <!-- opening on lower joint -->
+            <visual>
+                <origin xyz="0.024 0 -0.16" rpy="0 ${pi/2} 0" />
+                <geometry>
+                    <cylinder length="0.002" radius="0.014"/>
+                </geometry>
+                <material name="fingerpro_motor" />
+            </visual>
+        </link>
+        <joint name="finger_middle_to_motor_joint${suffix}" type="fixed">
+            <parent link="finger_middle_link${suffix}"/>
+            <child link="finger_middle_link_motor${suffix}"/>
+        </joint>
         <link name="finger_lower_link${suffix}">
             <xacro:add_geometry
@@ -85,5 +169,5 @@
                 xyz="0 0 0"
                 mesh_file="${lower_link_mesh}"
-                material="${material}"
+                material="fingerpro_shell"
                 mesh_scale="1."/>
             <xacro:add_inertia
@@ -100,5 +184,5 @@
                 xyz="-0.0185 0 ${lower_joint_to_tip_distance}"
                 mesh_file="${tip_link_mesh}"
-                material="${material}"
+                material="fingerpro_shell"
                 mesh_scale="1."/>
             <xacro:add_inertia

File: xacro/pro/trifingerpro.urdf.xacro (robot description, xacro)
@@ -4,15 +4,6 @@
     <xacro:include filename="fingerpro_macro.xacro" />
     <xacro:include filename="../macros.xacro" />
-    <material name="finger_0_material">
-        <color rgba="0.6 0.0 0.0 1.0" />
-    </material>
-    <material name="finger_120_material">
-        <color rgba="0.0 0.6 0.0 1.0" />
-    </material>
-    <material name="finger_240_material">
-        <color rgba="0.0 0.0 0.6 1.0" />
-    </material>
-    <material name="real_finger_material">
-        <color rgba="0.83 0.79 0.82 1.0" />
+    <material name="center_holder_material">
+        <color rgba="0.1 0.1 0.1 1.0" />
     </material>
     <!-- Define the global base_link and place all other objects relative to it. -->
@@ -32,5 +23,5 @@
             xyz="0 0 0"
             mesh_file="${center_link_mesh}"
-            material="real_finger_material"
+            material="center_holder_material"
             mesh_scale="1." />
         <!-- add inertial to suppress warning -->
@@ -48,7 +39,7 @@
     </joint>
     <!-- Define the three fingers and place them relative to the upper holder -->
-    <xacro:fingerpro suffix="_0" material="real_finger_material" />
-    <xacro:fingerpro suffix="_120" material="real_finger_material" />
-    <xacro:fingerpro suffix="_240" material="real_finger_material" />
+    <xacro:fingerpro suffix="_0" />
+    <xacro:fingerpro suffix="_120" />
+    <xacro:fingerpro suffix="_240" />
     <xacro:property name="angle_0" value="${radians(0)}"/>
     <xacro:property name="angle_120" value="${radians(120)}"/>
